File: Sensing subsystem/Schematic/Sensing systemv2/Sensing systemv2.kicad_sch (KiCad schematic)
At the start: 37 parts, among them J1 Conn_02x14_Odd_Even, Q1 SS8050

Commit message: Schematics
Parts:
- removed JP3, JP6, JP9: SoJMP_Opn3, Jumper:SolderJumper-3_P1.3mm_Open_RoundedPad1.0x1.5mm_NumberLabels, symbol Jumper:SolderJumper_3_Open
- removed R7: 10k, Resistor_SMD:R_0805_2012Metric, symbol Device:R_US
- added JP10, JP11, JP12, JP3, JP6, JP9: SoJMP_Opn, Jumper:SolderJumper-2_P1.3mm_Open_RoundedPad1.0x1.5mm, symbol Jumper:SolderJumper_2_Open
- added R17: 100k, Resistor_SMD:R_0805_2012Metric, symbol Device:R_US
- added R18: 12k, Resistor_SMD:R_0805_2012Metric, symbol Device:R_US
- added R19, R9: 10k, Resistor_SMD:R_0805_2012Metric, symbol Device:R_US
- D1, D2, D3, D4, D5, D6: footprint LED_THT:LED_D5.0mm -> LED_THT:LED_D5.0mm_Horizontal_O1.27mm_Z3.0mm_Clear
- J1: now not fitted
- R10, R16: value 100k -> 220k; LCSC C149504 -> C17556
- R11, R15, R5, R6: value 10k -> 220k; LCSC C17414 -> C17556; Price 0.0013 -> 0.0017
- R12: value 10k -> 100k; LCSC C17414 -> C149504; Price 0.0013 -> 0.0017
- R13: value 100k -> 12k; LCSC C149504 -> C17444
- R7: renamed from R9; value 10k -> 100k; LCSC C17414 -> C149504; Price 0.0013 -> 0.0017
- R8: value 10k -> 12k; LCSC C17414 -> C17444; Price 0.0013 -> 0.0017
- TP1, TP2, TP3, TP4: footprint TestPoint:TestPoint_Pad_2.0x2.0mm -> TestPoint:TestPoint_THTPad_D2.0mm_Drill1.0mm
Connections:
- net 3V3: now also JP1.1 (A), JP5.1 (A), R10.1, R15.1, R5.1, JP9.1 (A)
- net PA3: now also D6.1 (K), R15.2, R16.2, TP4.1, R17.2, R18.2, R19.2
- net PA4: now also D5.1 (K), R10.2, R11.2, R12.2, R13.2, R14.2, TP3.1; no longer D4.1 (K), R5.2, R7.2, R8.2, TP2.1
- net PA5: no longer D5.1 (K), R11.2, R12.2, R6.2, TP3.1
- net PA6: no longer D6.1 (K), R14.2, R15.2, TP4.1
- net PA7: now also D4.1 (K), R5.2, R6.2, R7.2, R8.2, TP2.1, R9.2
- net PE15: now also R4.1
- net PE8: no longer R4.1
- net at JP1.2 (B), JP2.1 (A): now also R6.1; no longer R10.2, R5.1
- net at R16.1: now also JP10.1 (A), JP9.2 (B)
- net at R11.1: now also JP5.2 (B), JP6.1 (A); no longer JP5.1 (A)
- net at R12.1: now also JP7.1 (A), JP6.2 (B); no longer JP4.2 (B)
- net at JP8.1 (A): now also JP7.2 (B), R13.1; no longer R14.1
- net at R8.1: now also JP4.1 (A), JP3.2 (B); no longer JP1.1 (A)
- net at JP2.2 (B), R7.1: now also JP3.1 (A)
- new net: JP10.2 (B), JP11.1 (A), R17.1
- new net: JP12.2 (B), R19.1
- new net: JP11.2 (B), JP12.1 (A), R18.1
- new net: JP8.2 (B), R14.1
- new net: JP4.2 (B), R9.1
Other:
- moved on the sheet: D5, D6, JP1, JP2, JP4, R7, TP3, TP4

Commit message: Sensing system
Connections:
- net PA3: now also D5.1 (K), R10.2, R11.2, R12.2, R13.2, R14.2, TP3.1; no longer D6.1 (K), R15.2, R16.2, R17.2, R18.2, R19.2, TP4.1
- net PA4: now also D6.1 (K), R15.2, R16.2, R17.2, R18.2, R19.2, TP4.1; no longer D5.1 (K), R10.2, R11.2, R12.2, R13.2, R14.2, TP3.1
Changed lines of the file:
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@@
 		)
 	)
-	(label "PA3"
+	(label "PA4"
 		(at 222.25 86.36 180)
 		(fields_autoplaced yes)
@@
 		)
 	)
-	(label "PA4"
+	(label "PA3"
 		(at 170.18 85.09 180)
 		(fields_autoplaced yes)
