File: Sensing subsystem/Schematic/Sensing systemv3/Sensing systemV3.kicad_sch (KiCad schematic)
At the start: 43 parts, among them J1 Conn_02x14_Odd_Even, Q1 SS8050

Commit message: Sensing system
Parts:
- J1: now fitted
- Q1: Populate (none) -> 1
- TP1, TP2, TP3, TP4: footprint TestPoint:TestPoint_THTPad_D2.0mm_Drill1.0mm -> TestPoint:TestPoint_Pad_2.0x2.0mm
