File: Sensing subsystem/Schematic/Sensing systemv3/_autosave-Sensing systemV3.kicad_sch (KiCad schematic)
At the start: 43 parts, among them J1 Conn_02x14_Odd_Even, Q1 SS8050

Commit message: Schematics
Other:
- note added: "Input"
- note added: "Out1"
- note added: "Out2"
- note added: "Out3"
Changed lines of the file:
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@@
+		)
+	)
+	(text "Out3"
+		(exclude_from_sim no)
+		(at 228.854 96.012 0)
+		(effects
+			(font
+				(size 1.27 1.27)
+			)
 		)
 	)
@@
 	(text "PE15 is connected to a PWM pin on the \nmicrocontroller to allow for switching \nand brightness control of the LEDs"
 		(exclude_from_sim no)
-		(at 23.368 106.426 0)
+		(at 23.368 109.474 0)
 		(effects
 			(font
@@
 				(thickness 1)
 				(bold yes)
+			)
+		)
+	)
+	(text "Input"
+		(exclude_from_sim no)
+		(at 67.056 102.87 0)
+		(effects
+			(font
+				(size 1.27 1.27)
 			)
 		)
@@
 		)
 	)
+	(text "Out2"
+		(exclude_from_sim no)
+		(at 176.53 94.996 0)
+		(effects
+			(font
+				(size 1.27 1.27)
+			)
+		)
+	)
 	(text "Left IR Emitter"
 		(exclude_from_sim no)
@@
 		(effects
 			(font
+				(size 1.27 1.27)
+			)
+		)
+	)
+	(text "Out1"
+		(exclude_from_sim no)
+		(at 125.73 92.202 0)
+		(effects
+			(font
