File: Power subsystem/Power Project PCB  v0/Power Project PCB  v0.kicad_sch (KiCad schematic)
At the start: 26 parts, among them J1 Conn_02x08_Even_Odd, J2 Conn_02x01, U1 MCP73831-2-OT, U2 DRV8837, U3 DRV8837

Commit message: pictures
Other:
- title: (none) -> EEE3088F Micromouse Power Subsystem Circuit
Changed lines of the file:
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@@
 	(generator_version "8.0")
 	(paper "A4")
+	(title_block
+		(title "EEE3088F Micromouse Power Subsystem Circuit")
+		(date "2024-03-24")
+		(rev "V0")
+		(comment 3 "ADMIMR011")
+		(comment 4 "Imran Adams")
+	)
 	(junction
 		(at 132.08 95.25)
